Commit message: Feat: Phase 1 Step 5 - Added parametric Lidar link and Gazebo sensor plugin

File: robo_swarm_description/urdf/mobile_base.xacro (robot description, xacro)
@@ -6,4 +6,6 @@
     <xacro:property name="wheel_radius" value="0.1" />
     <xacro:property name="wheel_length" value="0.05" />
+    <xacro:property name="lidar_radius" value ="0.05" />
+    <xacro:property name="lidar_height" value ="0.05" />
     <xacro:macro name="wheel_link" params="prefix">
         <link name="${prefix}_wheel_link">
@@ -61,4 +63,21 @@
         <xacro:sphere_inertia m="0.5" r="${wheel_radius/2.0}" o_xyz="0 0 0" o_rpy="0 0 0"/>
     </link>
+    <link name="lidar_link">
+        <visual>
+            <geometry>
+                <cylinder radius="${lidar_radius}" length="${lidar_height}" />
+            </geometry>
+            <material name="red">
+                <color rgba="1 0 0 1"/>
+            </material>
+        </visual>
+        <collision>
+            <geometry>
+                <cylinder radius="${lidar_radius}" length="${lidar_height}" />
+            </geometry>
+        </collision>
+        <xacro:cylinder_inertia m="0.1" r="${lidar_radius}" l="${lidar_height}"
+                             o_xyz="0 0 0" o_rpy="0 0 0"/>
+    </link>
     <joint name="base_foot_print_joint" type="fixed">
         <parent link="base_footprint"/>
@@ -83,3 +102,8 @@
         <origin xyz="${base_length/3.0} 0 ${-base_height/2.0 + wheel_radius/2.0}" rpy="0 0 0" />
     </joint>
+    <joint name="lidar_joint" type="fixed">
+        <parent link="base_link" />
+        <child link="lidar_link" />
+        <origin xyz="0 0 ${base_height + (lidar_height / 2.0)}" rpy="0 0 0" />
+    </joint>
 </robot>

File: robo_swarm_description/urdf/mobile_base_gazebo.xacro (robot description, xacro)
@@ -36,3 +36,28 @@
         </plugin>
     </gazebo>
+    <gazebo reference="lidar_link">
+        <sensor name="lidar" type="gpu_lidar">
+            <pose>0 0 0 0 0 0</pose>
+            <always_on>true</always_on>
+            <visualize>true</visualize>
+            <update_rate>10</update_rate>
+            <ray>
+                <scan>
+                    <horizontal>
+                        <samples>360</samples>
+                        <resolution>1</resolution>
+                        <min_angle>-3.14</min_angle>
+                        <max_angle>3.14</max_angle>
+                    </horizontal>
+                </scan>
+                <range>
+                    <min>0.3</min>
+                    <max>12</max>
+                </range>
+            </ray>
+            <plugin filename="gz-sim-sensors-system" name="gz::sim::systems::Sensors">
+                <render_engine>ogre2</render_engine>
+            </plugin>
+        </sensor>
+    </gazebo>
 </robot>
